File: BACEE.kicad_pcb (KiCad board)
At the start: 2 copper layers, 0 parts

Commit message: Set design rules.
Parts:
- added BT1: Battery 3V, Connector_PinHeader_2.54mm:PinHeader_1x02_P2.54mm_Vertical, F.Cu at (81.9, 85.7)
- added C1: 22 pF, Capacitor_SMD:C_0805_2012Metric_Pad1.18x1.45mm_HandSolder, F.Cu at (160.6, 107.2)
- added C2: 22 pF, Capacitor_SMD:C_0805_2012Metric_Pad1.18x1.45mm_HandSolder, F.Cu at (160.6, 110.2)
- added C3: 10 μF, Capacitor_SMD:C_0805_2012Metric_Pad1.18x1.45mm_HandSolder, F.Cu at (155.0, 114.4)
- added D1: LED, LED_SMD:LED_0805_2012Metric_Pad1.15x1.40mm_HandSolder, F.Cu at (155.0, 117.4)
- added J1: Serial Port, Connector_PinHeader_2.54mm:PinHeader_1x04_P2.54mm_Vertical, F.Cu at (91.1, 99.0)
- added J2: Digital pins, Connector_PinHeader_2.54mm:PinHeader_1x09_P2.54mm_Vertical, F.Cu at (81.8, 99.0)
- added J3: I2C, Connector_PinHeader_2.54mm:PinHeader_1x04_P2.54mm_Vertical, F.Cu at (86.5, 99.0)
- added J4: ISCP, Connector_PinHeader_2.54mm:PinHeader_2x03_P2.54mm_Vertical, F.Cu at (95.8, 99.0)
- added R1: 330 Ω, Resistor_SMD:R_0805_2012Metric_Pad1.20x1.40mm_HandSolder, F.Cu at (159.7, 117.4)
- added R2: 10K Ω, Resistor_SMD:R_0805_2012Metric_Pad1.20x1.40mm_HandSolder, F.Cu at (159.8, 114.4)
- added U1: 24LC1025, Package_SO:SOIJ-8_5.3x5.3mm_P1.27mm, F.Cu at (148.3, 104.3)
- added U2: DS1337S+, Package_SO:SO-8_5.3x6.2mm_P1.27mm, F.Cu at (147.4, 116.2)
- added U3: 24LC1025, Package_SO:SOIJ-8_5.3x5.3mm_P1.27mm, F.Cu at (136.9, 115.8)
- added U4: ATMEGA328-AU, digikey-footprints:TQFP-32_7x7mm, F.Cu at (137.3, 106.6)
- added Y1: Crystal 32MHz, Crystal:Crystal_SMD_MicroCrystal_CC7V-T1A-2Pin_3.2x1.5mm_HandSoldering, F.Cu at (146.4, 109.5)
- added Y2: Crystal 16MHz, Crystal:Crystal_SMD_5032-2Pin_5.0x3.2mm_HandSoldering, F.Cu at (158.7, 103.3)
Other:
- net class Power added: clearance 0.2, trace_width 0.3, via_dia 1, via_drill 0.6
